File: Locker/Locker.kicad_sch (KiCad schematic)
At the start: 6 parts, among them J1 GPIO, U1 CAT24C256

Commit message: /
Parts:
- removed C1: 100n, symbol Device:C_Small
- removed JP1: ID_WP, symbol Jumper:SolderJumper_2_Open
- removed R1, R2: 3.9k, symbol Device:R_Small
- removed U1: CAT24C256, symbol Memory_EEPROM:CAT24C256
- added Brd1: SSD1306, symbol SSD1306-128x64_OLED:SSD1306
- added C2: 10nF, symbol Device:C
- added C3: 47nF, symbol Device:C
- added J2: CRONA +9V, symbol something:Conn_01x02_Pin
- added J3, J4: SG90, symbol something:Conn_01x03_Pin_SG90
- added J6, J7: TCRT5000, symbol something:Conn_01x03_Pin_TCRT5000
- added J8, J9: KY-025, symbol something:Conn_01x04_Pin_KY-025
- added RFID1: RC522, symbol rc522:RC522
- added U2: L7805, symbol Regulator_Linear:L7805
Connections:
- net +3V3: now also Brd1.2 (VCC), J6.2 (VCC), J7.2 (VCC), J8.3 (VCC), J9.3 (VCC), RFID1.8 (3,3V)
- net GND: now also Brd1.1 (GND), C2.2, C3.2, J2.2 (GND), J4.1 (GND), J6.3 (GND), J7.3 (GND), J8.2 (GND), J9.2 (GND), RFID1.6 (GND), U2.2 (GND)
- net GPIO10/SPI0.MOSI: now also RFID1.3 (MOSI)
- net GPIO11/SPI0.SCLK: now also RFID1.2 (SCK)
- net GPIO17: now also J9.4 (D0)
- net GPIO22: now also J6.1 (S), RFID1.7 (RST)
- net GPIO23: now also J7.1 (S)
- net GPIO24: now also J3.3 (IN)
- net GPIO27: now also J8.4 (D0)
- net GPIO2/SDA1: now also Brd1.4 (SDA)
- net GPIO3/SCL1: now also Brd1.3 (SCL)
- net GPIO5: now also J4.3 (IN)
- net GPIO8/SPI0.CE0: now also RFID1.1 (SDA)
- net GPIO9/SPI0.MISO: now also RFID1.4 (MISO)
- new net: C2.1, J3.2 (VCC), J4.2 (VCC), U2.3 (OUT)
- new net: C3.1, J2.1 (+9V), U2.1 (IN)
- no-connect marks 3 -> 0
Other:
- note removed: "ID_SD and ID_SC PINS: These pins are reserved for HAT ID EEPROM. At boot time this I2C interface will be interrogated to look for an EEPROM that identifes the attached board and allows automagic setup of the GPIOs (and optionally, Linux drivers). Bridging JP1 enables write protection. DO NOT USE these pins for anything other than attaching an I2C ID EEPROM. Leave unconnected if ID EEPROM not requ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"
